Commit message: Co-authored-by:

File: assets/robots/hands/assembly_1/urdf/assembly_1_rotated.urdf (robot description, URDF)
Before this commit: robot assembly_1, 25 links, 24 joints
Joints:
- joint fixed_node_to_root_joint_0: origin xyz=0.0119296 0.00429764 -0.00662027 rpy=0 -0 0 -> xyz=0.00662027 -0.01192960 0.00429764 rpy=1.57079633 0.00000000 -1.57079633
